File: BleTouchDimmer/rf.sch (KiCad schematic (older format))
At the start: 7 parts

Commit message: Added component MDBT40.
Parts:
- gave numbers to parts that had none: 7
Changed lines of the file:
@@
 $EndDescr
 $Comp
-L C_Small C?
+L C_Small C10
 U 1 1 579681AC
 P 4200 3700
-F 0 "C?" H 4210 3770 50  0000 L CNN
+F 0 "C10" H 4210 3770 50  0000 L CNN
 F 1 "2n2" H 4210 3620 50  0000 L CNN
 F 2 "Capacitors_SMD:C_0805" H 4200 3700 50  0001 C CNN
@@
 $EndComp
 $Comp
-L L_Small L?
+L L_Small L2
 U 1 1 579681B3
 P 4200 3400
-F 0 "L?" H 4230 3440 50  0000 L CNN
+F 0 "L2" H 4230 3440 50  0000 L CNN
 F 1 "L_Small" H 4230 3360 50  0000 L CNN
 F 2 "" H 4200 3400 50  0000 C CNN
@@
 $EndComp
 $Comp
-L L_Small L?
+L L_Small L1
 U 1 1 579681BA
 P 4200 3100
-F 0 "L?" H 4230 3140 50  0000 L CNN
+F 0 "L1" H 4230 3140 50  0000 L CNN
 F 1 "L_Small" H 4230 3060 50  0000 L CNN
 F 2 "" H 4200 3100 50  0000 C CNN
@@
 $EndComp
 $Comp
-L C_Small C?
+L C_Small C11
 U 1 1 579681C1
 P 4550 2900
-F 0 "C?" H 4560 2970 50  0000 L CNN
+F 0 "C11" H 4560 2970 50  0000 L CNN
 F 1 "3p9" H 4560 2820 50  0000 L CNN
 F 2 "Capacitors_SMD:C_0805" H 4550 2900 50  0001 C CNN
@@
 $EndComp
 $Comp
-L C_Small C?
+L C_Small C12
 U 1 1 579681C8
 P 4750 3100
-F 0 "C?" H 4760 3170 50  0000 L CNN
+F 0 "C12" H 4760 3170 50  0000 L CNN
 F 1 "1p" H 4760 3020 50  0000 L CNN
 F 2 "Capacitors_SMD:C_0805" H 4750 3100 50  0001 C CNN
@@
 $EndComp
 $Comp
-L L_Small L?
+L L_Small L3
 U 1 1 579681CF
 P 4950 2900
-F 0 "L?" H 4980 2940 50  0000 L CNN
+F 0 "L3" H 4980 2940 50  0000 L CNN
 F 1 "L_Small" H 4980 2860 50  0000 L CNN
 F 2 "" H 4950 2900 50  0000 C CNN
@@
 Connection ~ 4200 3550
 $Comp
-L GND #PWR?
+L GND #PWR010
 U 1 1 57968CE9
 P 4200 3900
-F 0 "#PWR?" H 4200 3650 50  0001 C CNN
+F 0 "#PWR010" H 4200 3650 50  0001 C CNN
 F 1 "GND" H 4200 3750 50  0000 C CNN
 F 2 "" H 4200 3900 50  0000 C CNN
@@
 	4200 3800 4200 3900
 $Comp
-L C_Small C?
+L C_Small C13
 U 1 1 57969CD0
 P 5200 3100
-F 0 "C?" H 5210 3170 50  0000 L CNN
+F 0 "C13" H 5210 3170 50  0000 L CNN
 F 1 "1p5" H 5210 3020 50  0000 L CNN
 F 2 "Capacitors_SMD:C_0805" H 5200 3100 50  0001 C CNN
@@
 	5200 2900 5050 2900
 $Comp
-L GND #PWR?
+L GND #PWR011
 U 1 1 57969D53
 P 4750 3300
-F 0 "#PWR?" H 4750 3050 50  0001 C CNN
+F 0 "#PWR011" H 4750 3050 50  0001 C CNN
 F 1 "GND" H 4750 3150 50  0000 C CNN
 F 2 "" H 4750 3300 50  0000 C CNN
@@
 $EndComp
 $Comp
-L GND #PWR?
+L GND #PWR012
 U 1 1 57969D75
 P 5200 3300
-F 0 "#PWR?" H 5200 3050 50  0001 C CNN
+F 0 "#PWR012" H 5200 3050 50  0001 C CNN
 F 1 "GND" H 5200 3150 50  0000 C CNN
 F 2 "" H 5200 3300 50  0000 C CNN
