File: BleTouchDimmer/BleTouchDimmer.sch (KiCad schematic (older format))
At the start: 7 parts, among them U1 nRF51822, Y1 Crystal 16MHz, Y2 Crystal

Commit message: Started rf part.
Parts:
- added C?: 1n, symbol C
- added C? (x3): 100n, symbol C
- added C?: 47n, symbol C
- added R?: 10k, symbol R
- C3, C4: value 12pF -> 22pF
- Y2: footprint (none) -> EgertKiCad_lib:Crystal_ECX-31B; Ordering (none) -> http://www.mouser.ee/ProductDetail/ECS/ECS-327-125-34B-TR/?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
Connections:
- net labels added: +3.3V
- wire segments 25 -> 55
Other:
- note added: "712-ANT-2.45-CHP-T\nANT-2.54-CHP"
- note added: "Balun 497-13637-2-ND\nBAL-NRF01D3"
- moved on the sheet: C1, C2

Commit message: Added component MDBT40.
Parts:
- added U2: MDBT40, EgertKiCad_lib:MDBT40, symbol MDBT40
- gave numbers to parts that had none: 6
Changed lines of the file:
@@
 $EndComp
 $Comp
-L R R?
+L R R1
 U 1 1 57962E8D
 P 2450 2800
-F 0 "R?" V 2530 2800 50  0000 C CNN
+F 0 "R1" V 2530 2800 50  0000 C CNN
 F 1 "10k" V 2450 2800 50  0000 C CNN
 F 2 "" V 2380 2800 50  0000 C CNN
@@
 	2450 2550 2450 2650
 $Comp
-L GND #PWR?
+L GND #PWR03
 U 1 1 5796308D
 P 2450 3050
-F 0 "#PWR?" H 2450 2800 50  0001 C CNN
+F 0 "#PWR03" H 2450 2800 50  0001 C CNN
 F 1 "GND" H 2450 2900 50  0000 C CNN
 F 2 "" H 2450 3050 50  0000 C CNN
@@
 	2450 2950 2450 3050
 $Comp
-L GND #PWR?
+L GND #PWR04
 U 1 1 579637D7
 P 5550 5100
-F 0 "#PWR?" H 5550 4850 50  0001 C CNN
+F 0 "#PWR04" H 5550 4850 50  0001 C CNN
 F 1 "GND" H 5550 4950 50  0000 C CNN
 F 2 "" H 5550 5100 50  0000 C CNN
@@
 Connection ~ 5550 4750
 $Comp
-L +3.3V #PWR?
+L +3.3V #PWR05
 U 1 1 57963DF6
 P 5550 1500
-F 0 "#PWR?" H 5550 1350 50  0001 C CNN
+F 0 "#PWR05" H 5550 1350 50  0001 C CNN
 F 1 "+3.3V" H 5550 1640 50  0000 C CNN
 F 2 "" H 5550 1500 50  0000 C CNN
@@
 $EndComp
 $Comp
-L +3.3V #PWR?
+L +3.3V #PWR06
 U 1 1 5796402B
 P 3750 1700
-F 0 "#PWR?" H 3750 1550 50  0001 C CNN
+F 0 "#PWR06" H 3750 1550 50  0001 C CNN
 F 1 "+3.3V" H 3750 1840 50  0000 C CNN
 F 2 "" H 3750 1700 50  0000 C CNN
@@
 Connection ~ 3750 1950
 $Comp
-L C C?
+L C C9
 U 1 1 57964778
 P 5750 1550
-F 0 "C?" H 5775 1650 50  0000 L CNN
+F 0 "C9" H 5775 1650 50  0000 L CNN
 F 1 "1n" H 5775 1450 50  0000 L CNN
 F 2 "" H 5788 1400 50  0000 C CNN
@@
 Connection ~ 5550 1950
 $Comp
-L GND #PWR?
+L GND #PWR07
 U 1 1 5796534B
 P 6000 1600
-F 0 "#PWR?" H 6000 1350 50  0001 C CNN
+F 0 "#PWR07" H 6000 1350 50  0001 C CNN
 F 1 "GND" H 6000 1450 50  0000 C CNN
 F 2 "" H 6000 1600 50  0000 C CNN
@@
 	6000 1550 6000 1600
 $Comp
-L C C?
+L C C8
 U 1 1 57965937
 P 3500 2000
-F 0 "C?" H 3525 2100 50  0000 L CNN
+F 0 "C8" H 3525 2100 50  0000 L CNN
 F 1 "100n" H 3525 1900 50  0000 L CNN
 F 2 "" H 3538 1850 50  0000 C CNN
@@
 $EndComp
 $Comp
-L C C?
+L C C7
 U 1 1 57965994
 P 3200 2000
-F 0 "C?" H 3225 2100 50  0000 L CNN
+F 0 "C7" H 3225 2100 50  0000 L CNN
 F 1 "100n" H 3225 1900 50  0000 L CNN
 F 2 "" H 3238 1850 50  0000 C CNN
@@
 Connection ~ 3500 1750
 $Comp
-L GND #PWR?
+L GND #PWR08
 U 1 1 57965AD0
 P 3350 2200
-F 0 "#PWR?" H 3350 1950 50  0001 C CNN
+F 0 "#PWR08" H 3350 1950 50  0001 C CNN
 F 1 "GND" H 3350 2050 50  0000 C CNN
 F 2 "" H 3350 2200 50  0000 C CNN
@@
 Connection ~ 3350 2150
 $Comp
-L C C?
+L C C6
 U 1 1 57965DEF
 P 3100 3000
-F 0 "C?" H 3125 3100 50  0000 L CNN
+F 0 "C6" H 3125 3100 50  0000 L CNN
 F 1 "47n" H 3125 2900 50  0000 L CNN
 F 2 "" H 3138 2850 50  0000 C CNN
@@
 $EndComp
 $Comp
-L C C?
+L C C5
 U 1 1 57965E2E
 P 2850 3000
-F 0 "C?" H 2875 3100 50  0000 L CNN
+F 0 "C5" H 2875 3100 50  0000 L CNN
 F 1 "100n" H 2875 2900 50  0000 L CNN
 F 2 "" H 2888 2850 50  0000 C CNN
@@
 $EndComp
 $Comp
-L GND #PWR?
+L GND #PWR09
 U 1 1 57965E7C
 P 2850 3250
-F 0 "#PWR?" H 2850 3000 50  0001 C CNN
+F 0 "#PWR09" H 2850 3000 50  0001 C CNN
 F 1 "GND" H 2850 3100 50  0000 C CNN
 F 2 "" H 2850 3250 50  0000 C CNN
@@
 Text Notes 7450 2150 0    60   ~ 0
 712-ANT-2.45-CHP-T\nANT-2.54-CHP
+$Comp
+L MDBT40 U2
+U 1 1 5818CC93
+P 8650 4050
+F 0 "U2" H 7650 5000 60  0000 L CNN
+F 1 "MDBT40" H 8500 5000 60  0000 L CNN
+F 2 "EgertKiCad_lib:MDBT40" H 7450 4850 60  0001 C CNN
+F 3 "http://www.raytac.com/download/MDBT40/MDBT40%20spec-Version%20A4.pdf" H 7450 4850 60  0001 C CNN
+F 4 "http://www.ebay.com/itm/222215052092?_trksid=p2060353.m2749.l2649&ssPageName=STRK%3AMEBIDX%3AIT" H 8650 4050 60  0001 C CNN "Ordering"
+	1    8650 4050
+	1    0    0    -1
+$EndComp
 $EndSCHEMATC

Commit message: Removed nRF51 symbol.
Parts:
- removed C1, C2: 12pF, Capacitors_SMD:C_0805, symbol C
- removed C5, C8: 100n, symbol C
- removed U1: nRF51822, EgertKiCad_lib:QFN48N-NRF51822, symbol nRF51822
- removed Y1: Crystal 16MHz, Crystals:crystal_FA238-TSX3225, symbol Crystal
Connections:
- wire segments 55 -> 31
Other:
- note removed: "712-ANT-2.45-CHP-T\nANT-2.54-CHP"
- note removed: "Balun 497-13637-2-ND\nBAL-NRF01D3"
- moved on the sheet: C3, C4, C6, C7, C9, R1, U2

Commit message: Added uart, reset and programming part.
Parts:
- removed C6: 47n, symbol C
- added C1: 1n, Capacitors_SMD:C_0805, symbol C
- added P1: PROG, Socket_Strips:Socket_Strip_Straight_1x04, symbol CONN_01X04
- added P?: UART, Socket_Strips:Socket_Strip_Straight_1x04, symbol CONN_01X04
- added R2, R?: 10k, Resistors_SMD:R_0805, symbol R
- added SW1: SW_PUSH, Buttons_Switches_SMD:SW_SPST_B3SL-1022P, symbol SW_PUSH
- C7: value 100n -> 1u; footprint (none) -> Capacitors_SMD:C_0805
- C9: value 1n -> 1u; footprint (none) -> Capacitors_SMD:C_0805
- R1: footprint (none) -> Resistors_SMD:R_0805
Connections:
- net labels added: 3V3, RX, SWDCLK, SWDIO/RESET, TX
- wire segments 31 -> 53
- no-connect marks 0 -> 2
Other:
- note added: "PROG/DEBUG"
- note added: "UART"
- moved on the sheet: R1

Commit message: Updated RESET part.
Parts:
- added D?: LED, LEDs:LED_0805, symbol LED
- added R?: 100R, Resistors_SMD:R_0805, symbol R
- gave numbers to parts that had none: 2
Connections:
- wire segments 53 -> 57
Other:
- note added: "RESET"
- moved on the sheet: C1, R2, SW1
Changed lines of the file:
@@
 	3650 3550 3650 3600
 $Comp
-L GND #PWR01
+L GND #PWR2
 U 1 1 57955487
 P 3100 3950
-F 0 "#PWR01" H 3100 3700 50  0001 C CNN
+F 0 "#PWR2" H 3100 3700 50  0001 C CNN
 F 1 "GND" H 3100 3800 50  0000 C CNN
 F 2 "" H 3100 3950 50  0000 C CNN
@@
 $EndComp
 $Comp
-L GND #PWR02
+L GND #PWR4
 U 1 1 581A3066
 P 4250 2800
-F 0 "#PWR02" H 4250 2550 50  0001 C CNN
+F 0 "#PWR4" H 4250 2550 50  0001 C CNN
 F 1 "GND" H 4250 2650 50  0000 C CNN
 F 2 "" H 4250 2800 50  0000 C CNN
@@
 $EndComp
 $Comp
-L GND #PWR03
+L GND #PWR9
 U 1 1 581A31E1
 P 6950 2650
-F 0 "#PWR03" H 6950 2400 50  0001 C CNN
+F 0 "#PWR9" H 6950 2400 50  0001 C CNN
 F 1 "GND" H 6950 2500 50  0000 C CNN
 F 2 "" H 6950 2650 50  0000 C CNN
@@
 	3100 3850 3100 3950
 $Comp
-L GND #PWR04
+L GND #PWR5
 U 1 1 581A7CB9
 P 5000 4750
-F 0 "#PWR04" H 5000 4500 50  0001 C CNN
+F 0 "#PWR5" H 5000 4500 50  0001 C CNN
 F 1 "GND" H 5000 4600 50  0000 C CNN
 F 2 "" H 5000 4750 50  0000 C CNN
@@
 	5000 4550 5000 4750
 $Comp
-L GND #PWR05
+L GND #PWR8
 U 1 1 581A7D2A
 P 6200 4750
-F 0 "#PWR05" H 6200 4500 50  0001 C CNN
+F 0 "#PWR8" H 6200 4500 50  0001 C CNN
 F 1 "GND" H 6200 4600 50  0000 C CNN
 F 2 "" H 6200 4750 50  0000 C CNN
@@
 	6200 4550 6200 4750
 $Comp
-L GND #PWR06
+L GND #PWR7
 U 1 1 581A884C
 P 5000 5900
-F 0 "#PWR06" H 5000 5650 50  0001 C CNN
+F 0 "#PWR7" H 5000 5650 50  0001 C CNN
 F 1 "GND" H 5000 5750 50  0000 C CNN
 F 2 "" H 5000 5900 50  0000 C CNN
@@
 	5000 5800 5000 5900
 $Comp
-L GND #PWR07
+L GND #PWR1
 U 1 1 581ABEA9
 P 3100 3200
-F 0 "#PWR07" H 3100 2950 50  0001 C CNN
+F 0 "#PWR1" H 3100 2950 50  0001 C CNN
 F 1 "GND" H 3100 3050 50  0000 C CNN
 F 2 "" H 3100 3200 50  0000 C CNN
@@
 	3100 3100 3100 3200
 $Comp
-L +3.3V #PWR08
+L +3.3V #PWR6
 U 1 1 581AC6F3
 P 5000 5350
-F 0 "#PWR08" H 5000 5200 50  0001 C CNN
+F 0 "#PWR6" H 5000 5200 50  0001 C CNN
 F 1 "+3.3V" H 5000 5490 50  0000 C CNN
 F 2 "" H 5000 5350 50  0000 C CNN
@@
 Connection ~ 5000 5450
 $Comp
-L +3.3V #PWR09
+L +3.3V #PWR3
 U 1 1 581E4E9B
 P 3850 3050
-F 0 "#PWR09" H 3850 2900 50  0001 C CNN
+F 0 "#PWR3" H 3850 2900 50  0001 C CNN
 F 1 "+3.3V" H 3850 3190 50  0000 C CNN
 F 2 "" H 3850 3050 50  0000 C CNN
@@
 	7800 3850 7800 4000
 $Comp
-L GND #PWR010
+L GND #PWR10
 U 1 1 581AB091
 P 7800 4000
-F 0 "#PWR010" H 7800 3750 50  0001 C CNN
+F 0 "#PWR10" H 7800 3750 50  0001 C CNN
 F 1 "GND" H 7800 3850 50  0000 C CNN
 F 2 "" H 7800 4000 50  0000 C CNN
@@
 Text Label 7200 3250 0    60   ~ 0
 SWDCLK
-Wire Wire Line
-	6800 3350 8450 3350
 Text Label 7550 3350 2    60   ~ 0
 SWDIO/RESET
@@
 L R R2
 U 1 1 581E6B03
-P 8000 2900
-F 0 "R2" V 8080 2900 50  0000 C CNN
-F 1 "10k" V 8000 2900 50  0000 C CNN
-F 2 "Resistors_SMD:R_0805" V 7930 2900 50  0001 C CNN
-F 3 "" H 8000 2900 50  0000 C CNN
-	1    8000 2900
+P 9350 1050
+F 0 "R2" V 9430 1050 50  0000 C CNN
+F 1 "10k" V 9350 1050 50  0000 C CNN
+F 2 "Resistors_SMD:R_0805" V 9280 1050 50  0001 C CNN
+F 3 "" H 9350 1050 50  0000 C CNN
+	1    9350 1050
 	-1   0    0    1
 $EndComp
 $Comp
-L +3.3V #PWR011
+L +3.3V #PWR16
 U 1 1 581E6E36
-P 8000 2700
-F 0 "#PWR011" H 8000 2550 50  0001 C CNN
-F 1 "+3.3V" H 8000 2840 50  0000 C CNN
-F 2 "" H 8000 2700 50  0000 C CNN
-F 3 "" H 8000 2700 50  0000 C CNN
-	1    8000 2700
-	1    0    0    -1
-$EndComp
-Wire Wire Line
-	8000 3050 8000 3550
-Wire Wire Line
-	8000 2700 8000 2750
+P 9350 850
+F 0 "#PWR16" H 9350 700 50  0001 C CNN
+F 1 "+3.3V" H 9350 990 50  0000 C CNN
+F 2 "" H 9350 850 50  0000 C CNN
+F 3 "" H 9350 850 50  0000 C CNN
+	1    9350 850
+	1    0    0    -1
+$EndComp
+Wire Wire Line
+	9350 1200 9350 1700
+Wire Wire Line
+	9350 850  9350 900
 Wire Wire Line
 	7800 3250 7800 3550
@@
 L C C1
 U 1 1 581E7814
-P 8000 3700
-F 0 "C1" H 8025 3800 50  0000 L CNN
-F 1 "1n" H 8025 3600 50  0000 L CNN
-F 2 "Capacitors_SMD:C_0805" H 8038 3550 50  0001 C CNN
-F 3 "" H 8000 3700 50  0000 C CNN
-	1    8000 3700
+P 9350 1850
+F 0 "C1" H 9375 1950 50  0000 L CNN
+F 1 "1n" H 9375 1750 50  0000 L CNN
+F 2 "Capacitors_SMD:C_0805" H 9388 1700 50  0001 C CNN
+F 3 "" H 9350 1850 50  0000 C CNN
+	1    9350 1850
 	-1   0    0    1
 $EndComp
-Connection ~ 8000 3350
-Wire Wire Line
-	8000 3850 8000 3900
-Wire Wire Line
-	8000 3900 7800 3900
-Connection ~ 7800 3900
+Connection ~ 9350 1500
+Wire Wire Line
+	9350 2000 9350 2050
 $Comp
 L SW_PUSH SW1
 U 1 1 581E7B77
-P 8450 3750
-F 0 "SW1" H 8600 3860 50  0000 C CNN
-F 1 "SW_PUSH" H 8450 3670 50  0000 C CNN
-F 2 "Buttons_Switches_SMD:SW_SPST_B3SL-1022P" H 8450 3750 50  0001 C CNN
-F 3 "http://www.mouser.com/ds/2/15/SKQG-180836.pdf" H 8450 3750 50  0001 C CNN
-F 4 "http://www.mouser.ee/ProductDetail/ALPS/SKQGAKE010/?qs=sGAEpiMZZMsgGjVA3toVBA1UHfTHbV9%252bZVm6oBay0Ts%3d" H 8450 3750 60  0001 C CNN "Ordering"
-	1    8450 3750
+P 9800 1900
+F 0 "SW1" H 9950 2010 50  0000 C CNN
+F 1 "SW_PUSH" H 9800 1820 50  0000 C CNN
+F 2 "Buttons_Switches_SMD:SW_SPST_B3SL-1022P" H 9800 1900 50  0001 C CNN
+F 3 "http://www.mouser.com/ds/2/15/SKQG-180836.pdf" H 9800 1900 50  0001 C CNN
+F 4 "http://www.mouser.ee/ProductDetail/ALPS/SKQGAKE010/?qs=sGAEpiMZZMsgGjVA3toVBA1UHfTHbV9%252bZVm6oBay0Ts%3d" H 9800 1900 60  0001 C CNN "Ordering"
+	1    9800 1900
 	0    1    1    0
 $EndComp
 Wire Wire Line
-	8450 3350 8450 3450
-$Comp
-L GND #PWR012
+	9800 1500 9800 1600
+$Comp
+L GND #PWR18
 U 1 1 581E8389
-P 8450 4100
-F 0 "#PWR012" H 8450 3850 50  0001 C CNN
-F 1 "GND" H 8450 3950 50  0000 C CNN
-F 2 "" H 8450 4100 50  0000 C CNN
-F 3 "" H 8450 4100 50  0000 C CNN
-	1    8450 4100
-	1    0    0    -1
-$EndComp
-Wire Wire Line
-	8450 4050 8450 4100
+P 9800 2250
+F 0 "#PWR18" H 9800 2000 50  0001 C CNN
+F 1 "GND" H 9800 2100 50  0000 C CNN
+F 2 "" H 9800 2250 50  0000 C CNN
+F 3 "" H 9800 2250 50  0000 C CNN
+	1    9800 2250
+	1    0    0    -1
+$EndComp
+Wire Wire Line
+	9800 2200 9800 2250
 $Comp
 L CONN_01X04 P1
@@
 SWDIO/RESET
 $Comp
-L +3.3V #PWR013
+L +3.3V #PWR11
 U 1 1 581E9153
 P 9000 3200
-F 0 "#PWR013" H 9000 3050 50  0001 C CNN
+F 0 "#PWR11" H 9000 3050 50  0001 C CNN
 F 1 "+3.3V" H 9000 3340 50  0000 C CNN
 F 2 "" H 9000 3200 50  0000 C CNN
@@
 	9000 3200 9000 3250
 $Comp
-L GND #PWR014
+L GND #PWR12
 U 1 1 581E91BB
 P 9000 3600
-F 0 "#PWR014" H 9000 3350 50  0001 C CNN
+F 0 "#PWR12" H 9000 3350 50  0001 C CNN
 F 1 "GND" H 9000 3450 50  0000 C CNN
 F 2 "" H 9000 3600 50  0000 C CNN
@@
 PROG/DEBUG
 $Comp
-L CONN_01X04 P?
+L CONN_01X04 P2
 U 1 1 581EB0DF
 P 10250 4950
-F 0 "P?" H 10250 5200 50  0000 C CNN
+F 0 "P2" H 10250 5200 50  0000 C CNN
 F 1 "UART" V 10350 4950 50  0000 C CNN
 F 2 "Socket_Strips:Socket_Strip_Straight_1x04" H 10250 4950 50  0001 C CNN
@@
 TX
 $Comp
-L GND #PWR?
+L GND #PWR15
 U 1 1 581EB2A9
 P 9200 5150
-F 0 "#PWR?" H 9200 4900 50  0001 C CNN
+F 0 "#PWR15" H 9200 4900 50  0001 C CNN
 F 1 "GND" H 9200 5000 50  0000 C CNN
 F 2 "" H 9200 5150 50  0000 C CNN
@@
 	10050 4800 9200 4800
 $Comp
-L +3.3V #PWR?
+L +3.3V #PWR14
 U 1 1 581EB479
 P 9200 4750
-F 0 "#PWR?" H 9200 4600 50  0001 C CNN
+F 0 "#PWR14" H 9200 4600 50  0001 C CNN
 F 1 "+3.3V" H 9200 4890 50  0000 C CNN
 F 2 "" H 9200 4750 50  0000 C CNN
@@
 RX
 $Comp
-L R R?
+L R R3
 U 1 1 581ED91F
 P 9000 4700
-F 0 "R?" V 9080 4700 50  0000 C CNN
+F 0 "R3" V 9080 4700 50  0000 C CNN
 F 1 "10k" V 9000 4700 50  0000 C CNN
 F 2 "Resistors_SMD:R_0805" V 8930 4700 50  0001 C CNN
@@
 	9000 4850 9000 4900
 $Comp
-L +3.3V #PWR?
+L +3.3V #PWR13
 U 1 1 581EE473
 P 9000 4500
-F 0 "#PWR?" H 9000 4350 50  0001 C CNN
+F 0 "#PWR13" H 9000 4350 50  0001 C CNN
 F 1 "+3.3V" H 9000 4640 50  0000 C CNN
 F 2 "" H 9000 4500 50  0000 C CNN
@@
 Wire Notes Line
 	10450 4150 8750 4150
+Wire Wire Line
+	7550 3350 6800 3350
+Text Label 8650 1500 0    60   ~ 0
+SWDIO/RESET
+Wire Wire Line
+	8650 1500 9800 1500
+$Comp
+L GND #PWR17
+U 1 1 581EFF24
+P 9350 2050
+F 0 "#PWR17" H 9350 1800 50  0001 C CNN
+F 1 "GND" H 9350 1900 50  0000 C CNN
+F 2 "" H 9350 2050 50  0000 C CNN
+F 3 "" H 9350 2050 50  0000 C CNN
+	1    9350 2050
+	1    0    0    -1
+$EndComp
+Wire Notes Line
+	8450 600  8450 2550
+Wire Notes Line
+	8450 2550 10250 2550
+Wire Notes Line
+	10250 2550 10250 600
+Wire Notes Line
+	10250 600  8450 600
+Text Notes 8550 750  0    60   ~ 0
+RESET
+$Comp
+L R R?
+U 1 1 581F1BD4
+P 6900 4500
+F 0 "R?" V 6980 4500 50  0000 C CNN
+F 1 "100R" V 6900 4500 50  0000 C CNN
+F 2 "Resistors_SMD:R_0805" V 6830 4500 50  0001 C CNN
+F 3 "" H 6900 4500 50  0000 C CNN
+	1    6900 4500
+	-1   0    0    1
+$EndComp
+Wire Wire Line
+	6900 4350 6900 4250
+Wire Wire Line
+	6900 4250 6800 4250
+$Comp
+L LED D?
+U 1 1 581F1C9A
+P 6900 4950
+F 0 "D?" H 6900 5050 50  0000 C CNN
+F 1 "LED" H 6900 4850 50  0000 C CNN
+F 2 "LEDs:LED_0805" H 6900 4950 50  0001 C CNN
+F 3 "" H 6900 4950 50  0000 C CNN
+	1    6900 4950
+	0    -1   -1   0
+$EndComp
+Wire Wire Line
+	6900 4650 6900 4750
+$Comp
+L GND #PWR?
+U 1 1 581F1D57
+P 6900 5250
+F 0 "#PWR?" H 6900 5000 50  0001 C CNN
+F 1 "GND" H 6900 5100 50  0000 C CNN
+F 2 "" H 6900 5250 50  0000 C CNN
+F 3 "" H 6900 5250 50  0000 C CNN
+	1    6900 5250
+	1    0    0    -1
+$EndComp
+Wire Wire Line
+	6900 5150 6900 5250
 $EndSCHEMATC

Commit message: Started ZC_detect part. TODO select optoisolator.
Connections:
- net labels added: ZC_DETECT
- wire segments 57 -> 58
Changed lines of the file:
@@
 $Descr A4 11693 8268
 encoding utf-8
-Sheet 1 1
+Sheet 1 2
 Title ""
 Date ""
@@
 Wire Wire Line
 	6900 5150 6900 5250
+Wire Wire Line
+	5500 4550 5500 5250
+Text Label 5500 5250 1    60   ~ 0
+ZC_DETECT
+$Sheet
+S 5700 5750 900  550
+U 581F3B6C
+F0 "ZC_DETECT" 60
+F1 "ZC_DETECT.sch" 60
+$EndSheet
 $EndSCHEMATC

Commit message: Updated ZC part.
Parts:
- gave numbers to parts that had none: 2
Connections:
- wire segments 58 -> 61
- no-connect marks 2 -> 27
Changed lines of the file:
@@
 	3650 3550 3650 3600
 $Comp
-L GND #PWR2
+L GND #PWR01
 U 1 1 57955487
 P 3100 3950
-F 0 "#PWR2" H 3100 3700 50  0001 C CNN
+F 0 "#PWR01" H 3100 3700 50  0001 C CNN
 F 1 "GND" H 3100 3800 50  0000 C CNN
 F 2 "" H 3100 3950 50  0000 C CNN
@@
 $EndComp
 $Comp
-L GND #PWR4
+L GND #PWR02
 U 1 1 581A3066
 P 4250 2800
-F 0 "#PWR4" H 4250 2550 50  0001 C CNN
+F 0 "#PWR02" H 4250 2550 50  0001 C CNN
 F 1 "GND" H 4250 2650 50  0000 C CNN
 F 2 "" H 4250 2800 50  0000 C CNN
@@
 $EndComp
 $Comp
-L GND #PWR9
+L GND #PWR03
 U 1 1 581A31E1
 P 6950 2650
-F 0 "#PWR9" H 6950 2400 50  0001 C CNN
+F 0 "#PWR03" H 6950 2400 50  0001 C CNN
 F 1 "GND" H 6950 2500 50  0000 C CNN
 F 2 "" H 6950 2650 50  0000 C CNN
@@
 	3100 3850 3100 3950
 $Comp
-L GND #PWR5
+L GND #PWR04
 U 1 1 581A7CB9
 P 5000 4750
-F 0 "#PWR5" H 5000 4500 50  0001 C CNN
+F 0 "#PWR04" H 5000 4500 50  0001 C CNN
 F 1 "GND" H 5000 4600 50  0000 C CNN
 F 2 "" H 5000 4750 50  0000 C CNN
@@
 	5000 4550 5000 4750
 $Comp
-L GND #PWR8
+L GND #PWR05
 U 1 1 581A7D2A
 P 6200 4750
-F 0 "#PWR8" H 6200 4500 50  0001 C CNN
+F 0 "#PWR05" H 6200 4500 50  0001 C CNN
 F 1 "GND" H 6200 4600 50  0000 C CNN
 F 2 "" H 6200 4750 50  0000 C CNN
@@
 	6200 4550 6200 4750
 $Comp
-L GND #PWR7
+L GND #PWR06
 U 1 1 581A884C
 P 5000 5900
-F 0 "#PWR7" H 5000 5650 50  0001 C CNN
+F 0 "#PWR06" H 5000 5650 50  0001 C CNN
 F 1 "GND" H 5000 5750 50  0000 C CNN
 F 2 "" H 5000 5900 50  0000 C CNN
@@
 	5000 5800 5000 5900
 $Comp
-L GND #PWR1
+L GND #PWR07
 U 1 1 581ABEA9
 P 3100 3200
-F 0 "#PWR1" H 3100 2950 50  0001 C CNN
+F 0 "#PWR07" H 3100 2950 50  0001 C CNN
 F 1 "GND" H 3100 3050 50  0000 C CNN
 F 2 "" H 3100 3200 50  0000 C CNN
@@
 	3100 3100 3100 3200
 $Comp
-L +3.3V #PWR6
+L +3.3V #PWR08
 U 1 1 581AC6F3
 P 5000 5350
-F 0 "#PWR6" H 5000 5200 50  0001 C CNN
+F 0 "#PWR08" H 5000 5200 50  0001 C CNN
 F 1 "+3.3V" H 5000 5490 50  0000 C CNN
 F 2 "" H 5000 5350 50  0000 C CNN
@@
 Connection ~ 5000 5450
 $Comp
-L +3.3V #PWR3
+L +3.3V #PWR09
 U 1 1 581E4E9B
 P 3850 3050
-F 0 "#PWR3" H 3850 2900 50  0001 C CNN
+F 0 "#PWR09" H 3850 2900 50  0001 C CNN
 F 1 "+3.3V" H 3850 3190 50  0000 C CNN
 F 2 "" H 3850 3050 50  0000 C CNN
@@
 	7800 3850 7800 4000
 $Comp
-L GND #PWR10
+L GND #PWR010
 U 1 1 581AB091
 P 7800 4000
-F 0 "#PWR10" H 7800 3750 50  0001 C CNN
+F 0 "#PWR010" H 7800 3750 50  0001 C CNN
 F 1 "GND" H 7800 3850 50  0000 C CNN
 F 2 "" H 7800 4000 50  0000 C CNN
@@
 $EndComp
 $Comp
-L +3.3V #PWR16
+L +3.3V #PWR011
 U 1 1 581E6E36
 P 9350 850
-F 0 "#PWR16" H 9350 700 50  0001 C CNN
+F 0 "#PWR011" H 9350 700 50  0001 C CNN
 F 1 "+3.3V" H 9350 990 50  0000 C CNN
 F 2 "" H 9350 850 50  0000 C CNN
@@
 	9800 1500 9800 1600
 $Comp
-L GND #PWR18
+L GND #PWR012
 U 1 1 581E8389
 P 9800 2250
-F 0 "#PWR18" H 9800 2000 50  0001 C CNN
+F 0 "#PWR012" H 9800 2000 50  0001 C CNN
 F 1 "GND" H 9800 2100 50  0000 C CNN
 F 2 "" H 9800 2250 50  0000 C CNN
@@
 SWDIO/RESET
 $Comp
-L +3.3V #PWR11
+L +3.3V #PWR013
 U 1 1 581E9153
 P 9000 3200
-F 0 "#PWR11" H 9000 3050 50  0001 C CNN
+F 0 "#PWR013" H 9000 3050 50  0001 C CNN
 F 1 "+3.3V" H 9000 3340 50  0000 C CNN
 F 2 "" H 9000 3200 50  0000 C CNN
@@
 	9000 3200 9000 3250
 $Comp
-L GND #PWR12
+L GND #PWR014
 U 1 1 581E91BB
 P 9000 3600
-F 0 "#PWR12" H 9000 3350 50  0001 C CNN
+F 0 "#PWR014" H 9000 3350 50  0001 C CNN
 F 1 "GND" H 9000 3450 50  0000 C CNN
 F 2 "" H 9000 3600 50  0000 C CNN
@@
 TX
 $Comp
-L GND #PWR15
+L GND #PWR015
 U 1 1 581EB2A9
 P 9200 5150
-F 0 "#PWR15" H 9200 4900 50  0001 C CNN
+F 0 "#PWR015" H 9200 4900 50  0001 C CNN
 F 1 "GND" H 9200 5000 50  0000 C CNN
 F 2 "" H 9200 5150 50  0000 C CNN
@@
 	10050 4800 9200 4800
 $Comp
-L +3.3V #PWR14
+L +3.3V #PWR016
 U 1 1 581EB479
 P 9200 4750
-F 0 "#PWR14" H 9200 4600 50  0001 C CNN
+F 0 "#PWR016" H 9200 4600 50  0001 C CNN
 F 1 "+3.3V" H 9200 4890 50  0000 C CNN
 F 2 "" H 9200 4750 50  0000 C CNN
@@
 	9000 4850 9000 4900
 $Comp
-L +3.3V #PWR13
+L +3.3V #PWR017
 U 1 1 581EE473
 P 9000 4500
-F 0 "#PWR13" H 9000 4350 50  0001 C CNN
+F 0 "#PWR017" H 9000 4350 50  0001 C CNN
 F 1 "+3.3V" H 9000 4640 50  0000 C CNN
 F 2 "" H 9000 4500 50  0000 C CNN
@@
 	8650 1500 9800 1500
 $Comp
-L GND #PWR17
+L GND #PWR018
 U 1 1 581EFF24
 P 9350 2050
-F 0 "#PWR17" H 9350 1800 50  0001 C CNN
+F 0 "#PWR018" H 9350 1800 50  0001 C CNN
 F 1 "GND" H 9350 1900 50  0000 C CNN
 F 2 "" H 9350 2050 50  0000 C CNN
@@
 RESET
 $Comp
-L R R?
+L R R4
 U 1 1 581F1BD4
 P 6900 4500
-F 0 "R?" V 6980 4500 50  0000 C CNN
+F 0 "R4" V 6980 4500 50  0000 C CNN
 F 1 "100R" V 6900 4500 50  0000 C CNN
 F 2 "Resistors_SMD:R_0805" V 6830 4500 50  0001 C CNN
@@
 	6900 4250 6800 4250
 $Comp
-L LED D?
+L LED D1
 U 1 1 581F1C9A
 P 6900 4950
-F 0 "D?" H 6900 5050 50  0000 C CNN
+F 0 "D1" H 6900 5050 50  0000 C CNN
 F 1 "LED" H 6900 4850 50  0000 C CNN
 F 2 "LEDs:LED_0805" H 6900 4950 50  0001 C CNN
@@
 	6900 4650 6900 4750
 $Comp
-L GND #PWR?
+L GND #PWR019
 U 1 1 581F1D57
 P 6900 5250
-F 0 "#PWR?" H 6900 5000 50  0001 C CNN
+F 0 "#PWR019" H 6900 5000 50  0001 C CNN
 F 1 "GND" H 6900 5100 50  0000 C CNN
 F 2 "" H 6900 5250 50  0000 C CNN
@@
 ZC_DETECT
 $Sheet
-S 5700 5750 900  550
+S 5750 5650 900  550
 U 581F3B6C
 F0 "ZC_DETECT" 60
 F1 "ZC_DETECT.sch" 60
+F2 "ZC_DETECT" I L 5750 6050 60
+F3 "ZC_Line" I R 6650 5750 60
+F4 "ZC_N" I R 6650 5900 60
 $EndSheet
+Wire Wire Line
+	5200 6050 5750 6050
+Text Label 5200 6050 0    60   ~ 0
+ZC_DETECT
+$Comp
+L PWR_FLAG #FLG020
+U 1 1 581FAA9C
+P 7900 5650
+F 0 "#FLG020" H 7900 5745 50  0001 C CNN
+F 1 "PWR_FLAG" H 7900 5830 50  0000 C CNN
+F 2 "" H 7900 5650 50  0000 C CNN
+F 3 "" H 7900 5650 50  0000 C CNN
+	1    7900 5650
+	1    0    0    -1
+$EndComp
+$Comp
+L GND #PWR021
+U 1 1 581FAAED
+P 7900 5950
+F 0 "#PWR021" H 7900 5700 50  0001 C CNN
+F 1 "GND" H 7900 5800 50  0000 C CNN
+F 2 "" H 7900 5950 50  0000 C CNN
+F 3 "" H 7900 5950 50  0000 C CNN
+	1    7900 5950
+	1    0    0    -1
+$EndComp
+$Comp
+L +3.3V #PWR022
+U 1 1 581FAB37
+P 8450 5650
+F 0 "#PWR022" H 8450 5500 50  0001 C CNN
+F 1 "+3.3V" H 8450 5790 50  0000 C CNN
+F 2 "" H 8450 5650 50  0000 C CNN
+F 3 "" H 8450 5650 50  0000 C CNN
+	1    8450 5650
+	1    0    0    -1
+$EndComp
+$Comp
+L PWR_FLAG #FLG023
+U 1 1 581FAB81
+P 8450 5900
+F 0 "#FLG023" H 8450 5995 50  0001 C CNN
+F 1 "PWR_FLAG" H 8450 6080 50  0000 C CNN
+F 2 "" H 8450 5900 50  0000 C CNN
+F 3 "" H 8450 5900 50  0000 C CNN
+	1    8450 5900
+	-1   0    0    1
+$EndComp
+Wire Wire Line
+	8450 5650 8450 5900
+Wire Wire Line
+	7900 5650 7900 5950
+NoConn ~ 5300 4550
+NoConn ~ 5400 4550
+NoConn ~ 5600 4550
+NoConn ~ 5700 4550
+NoConn ~ 5800 4550
+NoConn ~ 5900 4550
+NoConn ~ 6000 4550
+NoConn ~ 6100 4550
+NoConn ~ 6800 2850
+NoConn ~ 6800 2950
+NoConn ~ 6800 3050
+NoConn ~ 6800 3150
+NoConn ~ 6800 3450
+NoConn ~ 6800 3550
+NoConn ~ 6800 3650
+NoConn ~ 6800 3950
+NoConn ~ 6800 4050
+NoConn ~ 6800 4150
+NoConn ~ 4400 4000
+NoConn ~ 4400 3900
+NoConn ~ 4400 3600
+NoConn ~ 4400 3500
+NoConn ~ 4400 3400
+NoConn ~ 4400 3300
+NoConn ~ 4400 3200
 $EndSCHEMATC

Commit message: Started Triac logic.
Parts:
- removed C1: 1n, Capacitors_SMD:C_0805, symbol C
- removed R2: 10k, Resistors_SMD:R_0805, symbol R
- removed SW1: SW_PUSH, Buttons_Switches_SMD:SW_SPST_B3SL-1022P, symbol SW_PUSH
Connections:
- wire segments 61 -> 59
Other:
- note removed: "RESET"
