File: BleTouchDimmer/_autosave-BleTouchDimmer.kicad_pcb (KiCad board)
At the start: 2 copper layers, 42 parts, among them P1 PROG, P2 UART, P3 POWER, Q1 PDTC123J, Q2 PDTC123J, SW1 SW_PUSH, U1 LTV-814, U2 MDBT40, U3 MOC3021S, U4 MOC3021S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

Commit message: Small changes.
Parts:
- added D5: Diode_Bridge, EgertKiCad_lib:SOIC-4, F.Cu at (106.4, 120.4)
- added U5: LNK4002S, TO_SOT_Packages_SMD:SOT-23-6, F.Cu at (144.5, 117.3)
- moved R20 94.5 mm to (185.4, 98.3)
- moved TR2 86.5 mm to (89.4, 137.2)
- moved P3 79.2 mm to (165.6, 122.4), turned to 0 degrees
- moved TR1 76.2 mm to (89.4, 121.9)
- moved U4 75.2 mm to (191.3, 87.9)
- moved Q2 66.3 mm to (194.3, 98.6)
- moved P1 54.7 mm to (132.6, 60.5)
- moved P2 47.5 mm to (125.0, 48.5), turned to 0 degrees
- moved U1 32.4 mm to (121.2, 116.1), turned to 90 degrees
- moved U3 31.6 mm to (159.3, 71.1)
- moved R3 11.6 mm to (99.6, 48.3)
- moved C9 7.12 mm to (116.1, 80.5)
- moved R2 7.12 mm to (116.6, 68.1)
- moved C7 7.12 mm to (116.3, 73.7)
