File: BleTouchDimmer/_autosave-BleTouchDimmer.kicad_pcb (KiCad board)
At the start: 2 copper layers, 50 parts, among them P1 PROG, P2 UART, P3 POWER, Q1 PDTC123J, Q2 PDTC123J, SW1 SW_PUSH, U1 LTV-814, U2 MDBT40, U3 MOC3021S, U4 MOC3021S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

Commit message: Started changing controller to esp32-wroom module.
Parts:
- removed C5: 1000uF, Capacitors_ThroughHole:C_Radial_D10_L13_P5
- added C2: 100n, Capacitors_SMD:C_0603, F.Cu at (81.9, 23.5)
- added U6: ESP32-WROOM, esp_library:ESP32-WROOM, F.Cu at (66.0, 52.1)
- added VR1: VR, Varistors:RV_Disc_D9_W4.4_P5, F.Cu at (108.0, 25.4)
- C6, C8: footprint Capacitors_SMD:C_0805 -> Capacitors_SMD:C_0603
- D1, D3, D4: footprint Resistors_SMD:R_0603_HandSoldering -> LEDs:LED_0805
- D6: footprint Resistors_SMD:R_0603_HandSoldering -> LEDs:LED_0603
- R21: footprint Resistors_SMD:R_0805 -> Resistors_SMD:R_0603
- U5: footprint SOT-223 -> TO_SOT_Packages_SMD:SOT-23-6
- moved C6 111.0 mm to (94.0, 18.4)
- moved C8 103.3 mm to (93.3, 30.5)
- moved D6 93.9 mm to (93.3, 30.5)
- moved R21 89.5 mm to (93.3, 30.5)
Connections:
- net /ZC_DETECT/ZC_DETECT renamed /ZC_DETECT
- P3 pad 2: (no net) -> /TR1_L_OUT
- P3 pad 3: (no net) -> /TR2_L_OUT
- P3 pad 4: (no net) -> /N
- Q1 pad 1: (no net) -> /TR1_CTRL
- Q2 pad 1: (no net) -> /TR2_CTRL
- R10 pad 1: (no net) -> /N
- R15 pad 2: /TRIACS/230VAC_L -> /230_VAC_L
- R17 pad 2: /TRIACS/230VAC_L -> /230_VAC_L
- R19 pad 2: /TRIACS/TRIAC1_L_OUT -> /TR1_L_OUT
- R20 pad 2: /TRIACS/TRIAC2_L_OUT -> /TR2_L_OUT
- R9 pad 1: (no net) -> /230_VAC_L
- TR1 pad 1: /TRIACS/TRIAC1_L_OUT -> /TR1_L_OUT
- TR1 pad 2: /TRIACS/230VAC_L -> /230_VAC_L
- TR2 pad 1: /TRIACS/TRIAC2_L_OUT -> /TR2_L_OUT
- TR2 pad 2: /TRIACS/230VAC_L -> /230_VAC_L
- TR3 pad 1: (no net) -> /230_VAC_L
- TR3 pad 5: (no net) -> /N
- U2 pad 27: (no net) -> /TR1_CTRL
- U2 pad 28: (no net) -> /TR2_CTRL
