File: BleTouchDimmer/TRIACS.sch (KiCad schematic (older format))
At the start: 5 parts, among them Q1 PDTC123J, U3 MOC3021S

Commit message: Changed MOC3021S footprint.
Parts:
- U3: footprint DIP-6 -> EgertKiCad_lib:MOC3021S
Other:
- note removed: "TODO Change footprint"
Changed lines of the file:
@@
 F 0 "U3" H 4640 3340 50  0000 L CNN
 F 1 "MOC3021S" H 4850 3350 50  0000 L CNN
-F 2 "DIP-6" H 4650 2950 50  0001 L CIN
+F 2 "EgertKiCad_lib:MOC3021S" H 4650 2950 50  0001 L CIN
 F 3 "http://www.mouser.com/ds/2/239/MOC302-201763.pdf" H 4825 3150 50  0001 L CNN
 F 4 "http://www.mouser.ee/ProductDetail/Lite-On/MOC3021S/?qs=sGAEpiMZZMteimceiIVCB9OIsGueWlCx1WN9Gn7xadE%3d" H 4850 3150 60  0001 C CNN "Source"
@@
 Wire Wire Line
 	3500 3500 3800 3500
-Text Notes 5250 3200 0    60   ~ 0
-TODO Change footprint
 $EndSCHEMATC

Commit message: Added triacs.
Parts:
- added D4: LED, LEDs:LED_0805, symbol LED
- added Q2: PDTC123J, TO_SOT_Packages_SMD:SOT-23, symbol DTC123J
- added R13: 100R, Resistors_SMD:R_0805, symbol R
- added R14: 220R, Resistors_SMD:R_0805, symbol R
- added R15, R16, R17, R18, R19, R20: 360R, Resistors_SMD:R_1206, symbol R
- added TR1, TR2: TRIAC, TO_SOT_Packages_SMD:TO-252-2Lead, symbol TRIAC
- added U4: MOC3021S, EgertKiCad_lib:MOC3021S, symbol MOC3021M
Connections:
- net labels added: 230VAC_L, TR1_CTRL, TR2_CTRL, TRIAC1_CONTROL, TRIAC1_L_OUT, TRIAC2_CONTROL, TRIAC2_L_OUT
- net labels removed: TRIAC_CONTROL
- wire segments 10 -> 40
Other:
- moved on the sheet: Q1, R11, R12, U3

Commit message: Updated power supply with LDO LD1117. TODO - Protection (VARISTOR, ??)
Parts:
- D3, D4: footprint LEDs:LED_0805 -> Resistors_SMD:R_0603_HandSoldering
Changed lines of the file:
@@
 $EndComp
 $Comp
-L GND #PWR25
+L GND #PWR026
 U 1 1 5821246B
 P 4200 3050
-F 0 "#PWR25" H 4200 2800 50  0001 C CNN
+F 0 "#PWR026" H 4200 2800 50  0001 C CNN
 F 1 "GND" H 4200 2900 50  0000 C CNN
 F 2 "" H 4200 3050 50  0000 C CNN
@@
 F 0 "D3" H 4200 2300 50  0000 C CNN
 F 1 "LED" H 4200 2100 50  0000 C CNN
-F 2 "LEDs:LED_0805" H 4200 2200 50  0001 C CNN
+F 2 "Resistors_SMD:R_0603_HandSoldering" H 4200 2200 50  0001 C CNN
 F 3 "" H 4200 2200 50  0000 C CNN
 	1    4200 2200
@@
 	4200 2400 4200 2500
 $Comp
-L +3V3 #PWR24
+L +3V3 #PWR027
 U 1 1 582125D3
 P 4200 1500
-F 0 "#PWR24" H 4200 1350 50  0001 C CNN
+F 0 "#PWR027" H 4200 1350 50  0001 C CNN
 F 1 "+3V3" H 4200 1640 50  0000 C CNN
 F 2 "" H 4200 1500 50  0000 C CNN
@@
 $EndComp
 $Comp
-L GND #PWR27
+L GND #PWR028
 U 1 1 58237C13
 P 4200 5750
-F 0 "#PWR27" H 4200 5500 50  0001 C CNN
+F 0 "#PWR028" H 4200 5500 50  0001 C CNN
 F 1 "GND" H 4200 5600 50  0000 C CNN
 F 2 "" H 4200 5750 50  0000 C CNN
@@
 F 0 "D4" H 4200 5000 50  0000 C CNN
 F 1 "LED" H 4200 4800 50  0000 C CNN
-F 2 "LEDs:LED_0805" H 4200 4900 50  0001 C CNN
+F 2 "Resistors_SMD:R_0603_HandSoldering" H 4200 4900 50  0001 C CNN
 F 3 "" H 4200 4900 50  0000 C CNN
 	1    4200 4900
@@
 	4200 5100 4200 5200
 $Comp
-L +3V3 #PWR26
+L +3V3 #PWR029
 U 1 1 58237C28
 P 4200 4200
-F 0 "#PWR26" H 4200 4050 50  0001 C CNN
+F 0 "#PWR029" H 4200 4050 50  0001 C CNN
 F 1 "+3V3" H 4200 4340 50  0000 C CNN
 F 2 "" H 4200 4200 50  0000 C CNN

Commit message: Uncommited changes.
Parts:
- D3, D4: footprint Resistors_SMD:R_0603_HandSoldering -> LEDs:LED_0603; symbol LED -> LED-RESCUE-BleTouchDimmer
- R11, R12, R13, R14: footprint Resistors_SMD:R_0805 -> Resistors_SMD:R_0603
Changed lines of the file:
@@
 EESchema Schematic File Version 2
+LIBS:BleTouchDimmer-rescue
+LIBS:cypress_touch
+LIBS:azoteq_touch
 LIBS:power
 LIBS:device
@@
 LIBS:Symbols_Microcontroller_Philips-NXP_RevA_06Oct2013
 LIBS:nordicsemi
-LIBS:Egert
 LIBS:Oscillators
 LIBS:74xgxx
@@
 LIBS:microchip_pic16mcu
 LIBS:microchip_pic18mcu
-LIBS:microchip_pic32mcu
 LIBS:motor_drivers
 LIBS:motors
@@
 LIBS:SymbolsSimilarEN60617+oldDIN617-RevE8
 LIBS:BleTouchDimmer-cache
-EELAYER 25 0
+EELAYER 26 0
 EELAYER END
 $Descr A4 11693 8268
@@
 F 0 "R11" V 4280 1750 50  0000 C CNN
 F 1 "100R" V 4200 1750 50  0000 C CNN
-F 2 "Resistors_SMD:R_0805" V 4130 1750 50  0001 C CNN
+F 2 "Resistors_SMD:R_0603" V 4130 1750 50  0001 C CNN
 F 3 "" H 4200 1750 50  0000 C CNN
 	1    4200 1750
@@
 $EndComp
 $Comp
-L LED D3
+L LED-RESCUE-BleTouchDimmer D3
 U 1 1 58212571
 P 4200 2200
+AR Path="/58212571" Ref="D3"  Part="1"
+AR Path="/58212355/58212571" Ref="D3"  Part="1"
 F 0 "D3" H 4200 2300 50  0000 C CNN
 F 1 "LED" H 4200 2100 50  0000 C CNN
-F 2 "Resistors_SMD:R_0603_HandSoldering" H 4200 2200 50  0001 C CNN
+F 2 "LEDs:LED_0603" H 4200 2200 50  0001 C CNN
 F 3 "" H 4200 2200 50  0000 C CNN
 	1    4200 2200
@@
 F 0 "R12" V 4580 1750 50  0000 C CNN
 F 1 "220R" V 4500 1750 50  0000 C CNN
-F 2 "Resistors_SMD:R_0805" V 4430 1750 50  0001 C CNN
+F 2 "Resistors_SMD:R_0603" V 4430 1750 50  0001 C CNN
 F 3 "" H 4500 1750 50  0000 C CNN
 	1    4500 1750
@@
 F 0 "R13" V 4280 4450 50  0000 C CNN
 F 1 "100R" V 4200 4450 50  0000 C CNN
-F 2 "Resistors_SMD:R_0805" V 4130 4450 50  0001 C CNN
+F 2 "Resistors_SMD:R_0603" V 4130 4450 50  0001 C CNN
 F 3 "" H 4200 4450 50  0000 C CNN
 	1    4200 4450
@@
 $EndComp
 $Comp
-L LED D4
+L LED-RESCUE-BleTouchDimmer D4
 U 1 1 58237C20
 P 4200 4900
+AR Path="/58237C20" Ref="D4"  Part="1"
+AR Path="/58212355/58237C20" Ref="D4"  Part="1"
 F 0 "D4" H 4200 5000 50  0000 C CNN
 F 1 "LED" H 4200 4800 50  0000 C CNN
-F 2 "Resistors_SMD:R_0603_HandSoldering" H 4200 4900 50  0001 C CNN
+F 2 "LEDs:LED_0603" H 4200 4900 50  0001 C CNN
 F 3 "" H 4200 4900 50  0000 C CNN
 	1    4200 4900
@@
 F 0 "R14" V 4580 4450 50  0000 C CNN
 F 1 "220R" V 4500 4450 50  0000 C CNN
-F 2 "Resistors_SMD:R_0805" V 4430 4450 50  0001 C CNN
+F 2 "Resistors_SMD:R_0603" V 4430 4450 50  0001 C CNN
 F 3 "" H 4500 4450 50  0000 C CNN
 	1    4500 4450
